File: ph-verzion-01.kicad_pcb (KiCad board)
At the start: 2 copper layers, 190 x 120 mm, 104 parts, among them J1 230V_IN, J10 OUT4, J11 AC_OUT_230V, J12 12V_IO, J2 DISPLAY, J3 1W_1, J4 1W_2, J5 1W_3, J6 1W_4, J7 GPIO_EXT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

Commit message: jedit
Parts:
- moved P2 26.9 mm to (183.0, 82.0)
- moved P1 25.3 mm to (183.0, 48.0)
- moved J12 24.7 mm to (68.0, 38.0)
- moved J1 24.5 mm to (35.0, 38.0)
- moved C11 23.3 mm to (158.0, 44.0)
- moved C12 23.3 mm to (158.0, 47.0)
- moved C15 23.3 mm to (162.0, 44.0)
- moved C16 23.3 mm to (162.0, 47.0)
- moved C17 23.3 mm to (162.0, 50.0)
- moved C8 22.4 mm to (82.0, 62.0)
- moved C22 21.9 mm to (162.0, 81.0)
- moved C23 21.9 mm to (162.0, 84.0)
- moved C24 21.9 mm to (162.0, 87.0)
- moved C26 21.2 mm to (165.0, 75.0)
- moved C27 21.2 mm to (165.0, 78.0)
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Other:
- board size 190 x 120 mm -> 160 x 100 mm

Commit message: opravy schemy
Parts:
- removed D7: M7, Diode_SMD:D_SMA
- added D8: PESD5V0S1BA, Diode_SMD:D_SOD-323, F.Cu at (147.9, 70.4)
- added D9: PESD5V0S1BA, Diode_SMD:D_SOD-323, F.Cu at (147.9, 73.3)
- added J13: PUMP, TerminalBlock_Phoenix:TerminalBlock_Phoenix_MKDS-1,5-2-5.08_1x02_P5.08mm_Horizontal, F.Cu at (114.9, 122.5)
- U6, U7, U8, U9: footprint Package_DIP:DIP-8_W7.62mm -> Package_SO:SOIC-8_3.9x4.9mm_P1.27mm
- moved U6 116.6 mm to (66.0, 125.8)
- moved C10 113.0 mm to (160.6, 151.0)
- moved U7 112.7 mm to (66.0, 132.4)
- moved R1 111.8 mm to (142.3, 132.8)
- moved C7 110.4 mm to (160.6, 135.3)
- moved MOV1 109.2 mm to (144.2, 44.9)
- moved C29 108.0 mm to (90.2, 150.0)
- moved J1 106.8 mm to (91.5, 128.7)
- moved J3 105.6 mm to (131.6, 120.8)
- moved J4 105.5 mm to (131.6, 128.6)
- moved J5 105.4 mm to (131.6, 136.4)
- moved J6 105.3 mm to (131.6, 144.2)
- moved U8 102.3 mm to (66.0, 139.0)
- moved U9 98.9 mm to (66.0, 145.6)
- moved C9 98.2 mm to (160.6, 143.1)
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Connections:
- D3 pad 1: +12V -> Net-(D3-K)
- D5 pad 1: +12V -> Net-(D5-K)
- D6 pad 1: +12V -> Net-(D6-K)
- J10 pad 2: +12V -> Net-(D6-K)
- J9 pad 2: +12V -> Net-(D5-K)
- Q1 pad 2: +12V -> Net-(D3-K)
- Q3 pad 2: +12V -> Net-(D5-K)
- Q4 pad 2: +12V -> Net-(D6-K)
- R11 pad 2: unconnected-(R11-Pad2) -> /ORP_CAL
- R15 pad 2: GND -> /ORP_CAL
- R4 pad 2: unconnected-(R4-Pad2) -> /pH_CAL
- R8 pad 2: GND -> /pH_CAL
- U10 pad 7: unconnected-(U10-AIN3-Pad7) -> GND
Other:
- board outline removed
- rule pad_to_mask_clearance: 0.1 -> 0
