File: oprava schemy - konektory a tak/ph-verzion-01.kicad_sch (KiCad schematic)
At the start: 106 parts, among them J1 230V_IN, J10 OUT4, J11 AC_OUT_230V, J12 12V_IO, J13 PUMP, J2 DISPLAY, J3 1W_1, J4 1W_2, J5 1W_3, J6 1W_4, J7 GPIO_EXT, J8 UART, J9 OUT3, P1 pH_BNC, P2 ORP_BNC, Q1 IRLR2905, Q2 IRLR2905, Q3 IRLR2905, Q4 IRLR2905, U1 HLK-30M12, U10 ADS1115, U11 ESP32-WROOM-32E-N4, U12 LTV-356T, U2 LM2596S-5.0, U3 LD1117AS33TR, U4 L7805ABD2T, U5 TPS60400, U6 CA3140EZ, U7 TL071IP, U8 CA3140EZ, U9 TL071IP

Commit message: opravy schemy
Changed lines of the file:
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@@
 	)
 	(junction
+		(at 124.9934 61.1886)
+		(diameter 0)
+		(color 0 0 0 0)
+	)
+	(junction
+		(at 124.9934 68.8086)
+		(diameter 0)
+		(color 0 0 0 0)
+	)
+	(junction
 		(at 54.991 109.9312)
 		(diameter 0)
@@
 	(wire
 		(pts
-			(xy 126.1872 59.9948) (xy 126.1872 64.9986)
+			(xy 126.1872 64.9986) (xy 126.1872 61.1886)
+		)
+		(stroke (width 0) (type default))
+	)
+	(wire
+		(pts
+			(xy 124.9934 61.1886) (xy 126.1872 61.1886)
+		)
+		(stroke (width 0) (type default))
+	)
+	(wire
+		(pts
+			(xy 126.1872 67.5386) (xy 126.1872 68.8086)
 		)
 		(stroke (width 0) (type default))
@@
 	(wire
 		(pts
-			(xy 126.1872 67.5386) (xy 126.1872 72.5424)
+			(xy 124.9934 68.8086) (xy 126.1872 68.8086)
 		)
 		(stroke (width 0) (type default))
@@
 	(wire
 		(pts
-			(xy 239.9284 222.5294) (xy 241.9096 222.5294)
+			(xy 239.9284 222.5294) (xy 249.9106 222.5294)
 		)
 		(stroke (width 0) (type default))
@@
 	(wire
 		(pts
-			(xy 276.098 193.2686) (xy 278.1046 193.2686)
+			(xy 276.098 193.2686) (xy 286.1056 193.2686)
 		)
 		(stroke (width 0) (type default))
@@
 	(wire
 		(pts
-			(xy 298.8818 189.992) (xy 300.8884 189.992)
+			(xy 298.8818 189.992) (xy 313.8932 189.992)
 		)
 		(stroke (width 0) (type default))
@@
 	(wire
 		(pts
-			(xy 239.9284 292.5318) (xy 241.9096 292.5318)
+			(xy 239.9284 292.5318) (xy 249.9106 292.5318)
 		)
 		(stroke (width 0) (type default))
@@
 	(wire
 		(pts
-			(xy 276.098 263.271) (xy 278.1046 263.271)
+			(xy 276.098 263.271) (xy 286.1056 263.271)
 		)
 		(stroke (width 0) (type default))
@@
 	(wire
 		(pts
-			(xy 298.8818 259.9944) (xy 300.8884 259.9944)
+			(xy 298.8818 259.9944) (xy 313.8932 259.9944)
 		)
 		(stroke (width 0) (type default))
@@
 	(wire
 		(pts
-			(xy 127.7874 267.1318) (xy 132.7912 267.1318)
+			(xy 127.7874 267.1318) (xy 142.7734 267.1318)
 		)
 		(stroke (width 0) (type default))
@@
 	(wire
 		(pts
-			(xy 127.7874 269.6718) (xy 132.7912 269.6718)
+			(xy 127.7874 269.6718) (xy 142.7734 269.6718)
 		)
 		(stroke (width 0) (type default))
@@
 	(wire
 		(pts
-			(xy 127.7874 272.2118) (xy 132.7912 272.2118)
+			(xy 127.7874 272.2118) (xy 142.7734 272.2118)
 		)
 		(stroke (width 0) (type default))
@@
 	(wire
 		(pts
-			(xy 127.7874 274.7518) (xy 132.7912 274.7518)
+			(xy 127.7874 274.7518) (xy 142.7734 274.7518)
 		)
 		(stroke (width 0) (type default))
@@
 	(wire
 		(pts
-			(xy 127.7874 277.2918) (xy 132.7912 277.2918)
+			(xy 127.7874 277.2918) (xy 142.7734 277.2918)
 		)
 		(stroke (width 0) (type default))
@@
 	(wire
 		(pts
-			(xy 127.7874 282.3718) (xy 132.7912 282.3718)
+			(xy 127.7874 282.3718) (xy 142.7734 282.3718)
 		)
 		(stroke (width 0) (type default))
@@
 	(wire
 		(pts
-			(xy 127.7874 284.9118) (xy 132.7912 284.9118)
+			(xy 127.7874 284.9118) (xy 142.7734 284.9118)
 		)
 		(stroke (width 0) (type default))
@@
 	(wire
 		(pts
-			(xy 127.7874 287.4518) (xy 132.7912 287.4518)
+			(xy 127.7874 287.4518) (xy 142.7734 287.4518)
 		)
 		(stroke (width 0) (type default))
@@
 	(wire
 		(pts
-			(xy 127.7874 289.9918) (xy 132.7912 289.9918)
+			(xy 127.7874 289.9918) (xy 142.7734 289.9918)
 		)
 		(stroke (width 0) (type default))
@@
 	(wire
 		(pts
-			(xy 127.7874 292.5318) (xy 132.7912 292.5318)
+			(xy 127.7874 292.5318) (xy 142.7734 292.5318)
 		)
 		(stroke (width 0) (type default))
@@
 	(wire
 		(pts
-			(xy 127.7874 295.0718) (xy 132.7912 295.0718)
+			(xy 127.7874 295.0718) (xy 142.7734 295.0718)
 		)
 		(stroke (width 0) (type default))
@@
 	(wire
 		(pts
-			(xy 127.7874 297.6118) (xy 132.7912 297.6118)
+			(xy 127.7874 297.6118) (xy 142.7734 297.6118)
 		)
 		(stroke (width 0) (type default))
@@
 	(wire
 		(pts
-			(xy 127.7874 300.1518) (xy 132.7912 300.1518)
+			(xy 127.7874 300.1518) (xy 142.7734 300.1518)
 		)
 		(stroke (width 0) (type default))
@@
 	(wire
 		(pts
-			(xy 127.7874 302.6918) (xy 132.7912 302.6918)
+			(xy 127.7874 302.6918) (xy 142.7734 302.6918)
 		)
 		(stroke (width 0) (type default))
@@
 	(wire
 		(pts
-			(xy 127.7874 305.2318) (xy 132.7912 305.2318)
+			(xy 127.7874 305.2318) (xy 142.7734 305.2318)
 		)
 		(stroke (width 0) (type default))
@@
 	(wire
 		(pts
-			(xy 127.7874 307.7718) (xy 132.7912 307.7718)
+			(xy 127.7874 307.7718) (xy 142.7734 307.7718)
 		)
 		(stroke (width 0) (type default))
@@
 	(wire
 		(pts
-			(xy 88.9 344.932) (xy 91.8972 344.932)
+			(xy 88.9 344.932) (xy 100.8888 344.932)
 		)
 		(stroke (width 0) (type default))
@@
 	(wire
 		(pts
-			(xy 140.1572 355.092) (xy 143.1544 355.092)
+			(xy 140.1572 355.092) (xy 152.1714 355.092)
 		)
 		(stroke (width 0) (type default))
@@
 	(wire
 		(pts
-			(xy 140.1572 344.932) (xy 143.1544 344.932)
+			(xy 140.1572 344.932) (xy 152.1714 344.932)
 		)
 		(stroke (width 0) (type default))
@@
 	)
 	(symbol
-		(lib_id "power:+12V")
-		(at 126.1872 59.9948 0)
-		(unit 1)
-		(exclude_from_sim no)
-		(in_bom yes)
-		(on_board yes)
-		(dnp no)
-		(property "Reference" "#PWR114" (at 128.7272 57.4548 0)
-			(effects (font (size 1.27 1.27)) (justify left))
-		)
-		(property "Value" "+12V" (at 128.7272 62.5348 0)
-			(effects (font (size 1.27 1.27)) (justify left))
-		)
-		(property "Footprint" "" (at 126.1872 59.9948 0)
-			(effects (font (size 1.27 1.27)) (hide yes))
-		)
-		(property "Datasheet" "~" (at 126.1872 59.9948 0)
-			(effects (font (size 1.27 1.27)) (hide yes))
-		)
-		(property "Description" "" (at 126.1872 59.9948 0)
-			(effects (font (size 1.27 1.27)) (hide yes))
-		)
-		(pin "1")
-		(instances
-			(project "ph-verzion-01"
-				(path "/54ccc777-3789-41c0-b4eb-6807475564db"
-					(reference "#PWR114")
-					(unit 1)
-				)
-			)
-		)
-	)
-	(symbol
-		(lib_id "power:GND")
-		(at 126.1872 72.5424 0)
-		(unit 1)
-		(exclude_from_sim no)
-		(in_bom yes)
-		(on_board yes)
-		(dnp no)
-		(property "Reference" "#PWR115" (at 128.7272 70.0024 0)
-			(effects (font (size 1.27 1.27)) (justify left))
-		)
-		(property "Value" "GND" (at 128.7272 75.0824 0)
-			(effects (font (size 1.27 1.27)) (justify left))
-		)
-		(property "Footprint" "" (at 126.1872 72.5424 0)
-			(effects (font (size 1.27 1.27)) (hide yes))
-		)
-		(property "Datasheet" "~" (at 126.1872 72.5424 0)
-			(effects (font (size 1.27 1.27)) (hide yes))
-		)
-		(property "Description" "" (at 126.1872 72.5424 0)
-			(effects (font (size 1.27 1.27)) (hide yes))
-		)
-		(pin "1")
-		(instances
-			(project "ph-verzion-01"
-				(path "/54ccc777-3789-41c0-b4eb-6807475564db"
-					(reference "#PWR115")
-					(unit 1)
-				)
-			)
-		)
-	)
-	(symbol
 		(lib_id "Device:R")
 		(at 140.0048 62.0014 0)
@@
 		(on_board yes)
 		(dnp no)
-		(property "Reference" "#PWR111" (at 217.551 206.4512 0)
+		(property "Reference" "#PWR101" (at 217.551 206.4512 0)
 			(effects (font (size 1.27 1.27)) (justify left))
 		)
@@
 			(project "ph-verzion-01"
 				(path "/54ccc777-3789-41c0-b4eb-6807475564db"
-					(reference "#PWR111")
+					(reference "#PWR101")
 					(unit 1)
 				)
@@
 		(on_board yes)
 		(dnp no)
-		(property "Reference" "#PWR112" (at 217.551 276.4536 0)
+		(property "Reference" "#PWR102" (at 217.551 276.4536 0)
 			(effects (font (size 1.27 1.27)) (justify left))
 		)
@@
 			(project "ph-verzion-01"
 				(path "/54ccc777-3789-41c0-b4eb-6807475564db"
-					(reference "#PWR112")
+					(reference "#PWR102")
 					(unit 1)
 				)
@@
 		(on_board yes)
 		(dnp no)
-		(property "Reference" "#PWR113" (at 338.582 197.4596 0)
+		(property "Reference" "#PWR100" (at 338.582 197.4596 0)
 			(effects (font (size 1.27 1.27)) (justify left))
 		)
@@
 			(project "ph-verzion-01"
 				(path "/54ccc777-3789-41c0-b4eb-6807475564db"
-					(reference "#PWR113")
+					(reference "#PWR100")
 					(unit 1)
 				)
