File: pred routingom/ph-verzion-01.kicad_pcb (KiCad board)
At the start: 2 copper layers, 114.5 x 148.5 mm, 106 parts, among them J1 230V_IN, J10 OUT4, J11 AC_OUT_230V, J12 12V_IO, J13 PUMP, J2 DISPLAY, J3 1W_1, J4 1W_2, J5 1W_3, J6 1W_4, J7 GPIO_EXT, J8 UART, J9 OUT3, P1 pH_BNC, P2 ORP_BNC, Q1 IRLR2905, Q2 IRLR2905, Q3 IRLR2905, Q4 IRLR2905, U1 HLK-30M12, U10 ADS1115, U11 ESP32-WROOM-32E-N4, U12 LTV-356T, U2 LM2596S-5.0, U3 LD1117AS33TR, U4 L7805ABD2T, U5 TPS60400, U6 CA3140EZ, U7 TL071IP, U8 CA3140EZ, U9 TL071IP

Commit message: uprava dosky pred routingom
Other:
- board outline removed
Changed lines of the file:
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@@
 	)
 	(setup
-		(stackup
-			(layer "F.SilkS"
-				(type "Top Silk Screen")
-			)
-			(layer "F.Paste"
-				(type "Top Solder Paste")
-			)
-			(layer "F.Mask"
-				(type "Top Solder Mask")
-				(thickness 0.01)
-			)
-			(layer "F.Cu"
-				(type "copper")
-				(thickness 0.035)
-			)
-			(layer "dielectric 1"
-				(type "core")
-				(thickness 1.51)
-				(material "FR4")
-				(epsilon_r 4.5)
-				(loss_tangent 0.02)
-			)
-			(layer "B.Cu"
-				(type "copper")
-				(thickness 0.035)
-			)
-			(layer "B.Mask"
-				(type "Bottom Solder Mask")
-				(thickness 0.01)
-			)
-			(layer "B.Paste"
-				(type "Bottom Solder Paste")
-			)
-			(layer "B.SilkS"
-				(type "Bottom Silk Screen")
-			)
-			(copper_finish "None")
-			(dielectric_constraints no)
-		)
 		(pad_to_mask_clearance 0)
 		(allow_soldermask_bridges_in_footprints no)
@@
 		(capping no)
 		(filling no)
-		(zone_defaults)
 		(pcbplotparams
 			(layerselection 0x00000000_00000000_55555555_5755f5ff)
@@
 		)
 	)
-	(gr_poly
-		(pts
-			(xy 23 22.5) (xy 23.5 170.5) (xy 137 170.5) (xy 137.5 22) (xy 23 22)
-		)
-		(stroke
-			(width 0.05)
-			(type solid)
-		)
-		(fill no)
-		(layer "Edge.Cuts")
-	)
 	(embedded_fonts no)
